File: Controller.kicad_pcb (KiCad board)
At the start: 2 copper layers, 21 parts, among them J1 ToArduino, J2 FromArduino, J3 Power12V, J4 A0 Sensor, J5 D12, J6 D4 - Heat, J7 D11, J8 D5-Fan, Q1 IRF-Heat, Q2 IRF-Fan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

Commit message: version 1.1 #4 #5
Parts:
- D1: footprint Diode_THT:D_DO-15_P15.24mm_Horizontal -> Diode_THT:D_DO-15_P5.08mm_Vertical_KathodeUp
- moved Q2 13.5 mm to (122.6, 44.5), turned to 270 degrees
- moved J8 9.44 mm to (104.1, 45.0)
- moved J6 9.14 mm to (80.6, 44.8)
- moved D1 6.36 mm to (118.6, 45.1)
- moved R8 5.84 mm to (108.8, 47.2)
- moved R5 5.59 mm to (86.7, 44.6)
- moved Q1 4.99 mm to (92.7, 45.3)
Connections:
- J1 pad 1: Net-(J1-Pad1) -> Net-(D1-Pad2)
- J3 pad 2: Net-(J1-Pad1) -> Net-(D1-Pad2)
- Q1 pad 2: Net-(D1-Pad2) -> Net-(Q1-Pad2)
- R5 pad 1: Net-(D1-Pad2) -> Net-(Q1-Pad2)
- R5 pad 2: Net-(J1-Pad1) -> Net-(D1-Pad2)
Routing:
- net Net-(J8-Pad1): track 12.8 -> 37.2 mm
- net Net-(J1-Pad1): track 22.6 -> 0.00 mm
- net Net-(D1-Pad2): track 39.7 -> 61.4 mm
- net Net-(Q1-Pad2): track 0.00 -> 9.57 mm
- net Net-(J6-Pad1): track 13.9 -> 22.8 mm
- net Net-(D1-Pad1): track 26.7 -> 23.5 mm
- net Net-(J2-Pad2): track 94.6 -> 96.6 mm
Other:
- board text added: "Incubator BioLab"
- board text added: "based on"
- board text added: "https://www.instructables.com/Incubadora-Garagem-FabLab-Biohackacademy/"
